File: Eagle Design/CC3200_Breakout.sch (EAGLE design)
At the start: 49 parts, among them Y1 32.768KHz, Y2 407MHz

Commit message: BRD and name
Rename the component on schema to match name with LaunchPad XL and added
first BRD file with component placement only
Parts:
- removed C21: 0.1uF, resistor:C-USC0402K
- removed C6, C7: 100uF, resistor:C-USC0402K
- removed Y1: 32.768KHz, SparkFun-FreqCtrl:CRYSTAL5X3
- added C30: 0.1uF, resistor:C-USC0402K
- added C47, C48: 6.2pF, resistor:C-USC0402K
- added Y3: 407MHz, SparkFun-FreqCtrl:CRYSTAL5X3
- C23: value 0.1uF -> 100uF
- C24: value 10pF -> 100uF
- C26: value 6.2pF -> 10pF
- C27: value 6.2pF -> 10uF
- C50: value (none) -> 1.0pF
- Y2: value 407MHz -> 32.768KHz
- renumbered $FL1 to FL1, C1 to C40, C10 to C41, C11 to C31, C12 to C35, C13 to C43, C14 to C45, C15 to C34, C16 to C36, C17 to C42, C18 to C32, C19 to C37, C2 to C38, C20 to C28, C22 to C44, C3 to C33, C4 to C29, C5 to C39, C9 to C50, L1 to L7, L2 to L6, L3 to L5, L4 to L9, R10 to R61, R5 to R64, R7 to R65, R8 to R58, R9 to R59, U$2 to U15
Connections:
- net N$23 renamed JTAG_TDO
- net N$24 renamed JTAG_TDI
- net N$25 renamed JTAG_TMS
- net N$26 renamed JTAG_TCK
- net GND: now also C30.2, C47.2, C48.2; no longer C21.2, C6.2, C7.2
- net N$1: now also C26.1, Y2.2; no longer C24.1, Y1.2
- net N$18: now also C30.1; no longer C23.1
- net N$2: now also Y2.1; no longer Y1.1
- net N$20: now also C27.1; no longer C21.1
- net N$28: now also C47.1, Y3.2; no longer C26.1, Y2.2
- net N$29: now also C48.1, Y3.1; no longer C27.1, Y2.1
- net V_BATT: now also C23.1, C24.1; no longer C6.1, C7.1
Other:
- moved on the sheet: C23, C24, C26, C27, Y2

Commit message: Some placement and renaming
Removed Pull up and Pull down from Flash Chip and rename SPI pins
Parts:
- removed R2, R3, R4: 100k, resistor:R-US_R0402
- removed U$4, U$5: M10X2, SparkFun-Connectors:M10X2
- added J22, J23: M10X2, SparkFun-Connectors:M10X2
Connections:
- removed net 1: U$1.GPIO_10, U$4.17
- removed net 2: U$1.GPIO_11, U$4.19
- removed net 5: U$1.GPIO_14, U$4.13
- removed net 6: U$1.GPIO_15, U$5.14
- removed net 7: U$1.GPIO_16, U$5.12
- removed net 8: U$1.GPIO_17, U$5.6
- removed net N$15: U$4.1
- removed net N$77: U$4.2
- removed net N$78: U$4.4
- new net SCL: J22.17, U$1.GPIO_10
- new net SDA: J22.19, U$1.GPIO_11
- new net SPI_CLK: J22.13, U$1.GPIO_14
- new net SPI_CS: J23.6, U$1.GPIO_17
- new net SPI_MISO: J23.14, U$1.GPIO_15
- new net SPI_MOSI: J23.12, U$1.GPIO_16
- new net VCC_BRD: J22.1
- new net VCC_MCU_5V: J22.2
- net 15: now also J23.20; no longer U$5.20
- net 16: now also J23.17; no longer U$5.17
- net 17: now also J23.19; no longer U$5.19
- net 18: now also J23.4; no longer U$5.4
- net 21: now also J23.16; no longer U$5.16
- net 3: now also J22.7; no longer U$4.7
- net 4: now also J22.5; no longer U$4.5
- net 45: now also J23.8; no longer U$5.8
- net 50: now also J22.20; no longer U$4.20
- net 53: now also J22.16; no longer U$4.16
- net 55: now also J23.18; no longer U$5.18
- net 57: now also J22.6; no longer U$4.6
- net 58: now also J22.3; no longer U$4.3
- net 59: now also J22.11; no longer U$4.11
- net 60: now also J22.8; no longer U$4.8
- net 61: now also J22.9; no longer U$4.9
- net 62: now also J22.15; no longer U$4.15
- net 63: now also J22.14; no longer U$4.14
- net 64: now also J22.18; no longer U$4.18
- net GND: now also J22.4, J23.2; no longer R3.1, R4.1, U$5.2
- net N$30: no longer R2.2
- net N$32: no longer R4.2
- net N$33: no longer R3.2
- net N$47: now also J23.1; no longer U$5.1
- net N$48: now also J23.3; no longer U$5.3
- net N$49: now also J23.5; no longer U$5.5
- net N$50: now also J23.7; no longer U$5.7
- net N$51: now also J23.9; no longer U$5.9
- net N$52: now also J23.11; no longer U$5.11
- net N$53: now also J23.13; no longer U$5.13
- net N$54: now also J23.15; no longer U$5.15
- net N$81: now also J22.10; no longer U$4.10
- net N$82: now also J22.12; no longer U$4.12
- net N$91: now also J23.10; no longer U$5.10
- net V_BATT: no longer R2.1
